File: hw.brd (EAGLE design)
At the start: 52.2 x 43.2 mm, 75 parts, among them IC1 ATMEGA32U4-AU, IC2 LTC485S, IC3 MCP16301/H, IC5 DS18S20, J1 Temperature sensor, J2 Flow sensor, J3 Level sensor, Q1 GSX-533, SW1 SPS, SW2 SPS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

Commit message: Changed library of crystal
Parts:
- Q1: device GSX-533:5032 -> crystal-golledge:5032
Changed lines of the file:
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@@
 <attribute name="VALUE" x="0.3225" y="24.4" size="1.016" layer="28" rot="MR90"/>
 </element>
-<element name="Q1" library="GSX-533" package="5032" value="GSX-533" x="22.86" y="13.335" rot="MR270"/>
+<element name="Q1" library="crystal-golledge" library_urn="urn:adsk.eagle:library:4881003" package="5032" package3d_urn="urn:adsk.eagle:package:4881006/2" value="GSX-533" x="22.86" y="13.335" rot="MR270"/>
 </elements>
 <signals>
